File: Ports.sch (KiCad schematic (older format))
At the start: 45 parts, among them J4 Conn_01x04_Male, J5 Conn_01x04_Male, J6 Conn_01x04_Male, J7 Conn_01x04_Male, J8 Conn_01x04_Male, Q10 BSS138, Q5 BSS138, Q6 BSS138, Q8 BSS138

Commit message: Add files via upload
Parts:
- added H1, H2, H3, H4: MountingHole, MountingHole:MountingHole_3.2mm_M3, symbol Mechanical:MountingHole
- D10, D11, D12, D13, D16, D17, D18, D19, D8, D9: footprint (none) -> Package_TO_SOT_SMD:SOT-323_SC-70; symbol BAT30S:D_BAT30S -> SAM21-rescue:D_BAT30S-BAT30S
- D22, D23: symbol DMP1045U:DMP1045U -> SAM21-rescue:DMP1045U-DMP1045U
Connections:
- net GND: now also D8.1 (A)
- net D10_TX11.5B renamed D10_TX13.2C
- net D11_RX11.5C renamed D11_RX13.2C
- net D12_TX21.5C renamed D12_TX23.3C
- net D13_TX21.5C renamed D13_RX23.3C
- net D14_I2C_PWR1.5C renamed D14_I2C_PWR3.5B
- net D15_SDA1.5B renamed D15_SDA3.5B
- net D16_SCL1.5B renamed D16_SCL3.5B
- net D9_UART_PWR1.5C renamed D9_UART_PWR3.1D
Changed lines of the file:
@@
 	3400 2600 3000 2600
 $Comp
-L BAT30S:D_BAT30S D9
+L SAM21-rescue:D_BAT30S-BAT30S D9
 U 1 1 5D647358
 P 5350 1950
 F 0 "D9" H 5172 2071 50  0000 R CNN
 F 1 "D_BAT30S" H 5172 1980 50  0000 R CNN
-F 2 "" H 5350 1950 50  0001 C CNN
+F 2 "Package_TO_SOT_SMD:SOT-323_SC-70" H 5350 1950 50  0001 C CNN
 F 3 "" H 5350 1950 50  0001 C CNN
 	1    5350 1950
@@
 $EndComp
 $Comp
-L BAT30S:D_BAT30S D10
+L SAM21-rescue:D_BAT30S-BAT30S D10
 U 1 1 5D6487EE
 P 6000 1950
 F 0 "D10" H 5822 2071 50  0000 R CNN
 F 1 "D_BAT30S" H 5822 1980 50  0000 R CNN
-F 2 "" H 6000 1950 50  0001 C CNN
+F 2 "Package_TO_SOT_SMD:SOT-323_SC-70" H 6000 1950 50  0001 C CNN
 F 3 "" H 6000 1950 50  0001 C CNN
 	1    6000 1950
@@
 $EndComp
 $Comp
-L BAT30S:D_BAT30S D12
+L SAM21-rescue:D_BAT30S-BAT30S D12
 U 1 1 5D6490F9
 P 7250 1950
 F 0 "D12" H 7072 2071 50  0000 R CNN
 F 1 "D_BAT30S" H 7072 1980 50  0000 R CNN
-F 2 "" H 7250 1950 50  0001 C CNN
+F 2 "Package_TO_SOT_SMD:SOT-323_SC-70" H 7250 1950 50  0001 C CNN
 F 3 "" H 7250 1950 50  0001 C CNN
 	1    7250 1950
@@
 $EndComp
 $Comp
-L BAT30S:D_BAT30S D13
+L SAM21-rescue:D_BAT30S-BAT30S D13
 U 1 1 5D6494B0
 P 7900 1950
 F 0 "D13" H 7722 2071 50  0000 R CNN
 F 1 "D_BAT30S" H 7722 1980 50  0000 R CNN
-F 2 "" H 7900 1950 50  0001 C CNN
+F 2 "Package_TO_SOT_SMD:SOT-323_SC-70" H 7900 1950 50  0001 C CNN
 F 3 "" H 7900 1950 50  0001 C CNN
 	1    7900 1950
@@
 $EndComp
 $Comp
-L BAT30S:D_BAT30S D8
+L SAM21-rescue:D_BAT30S-BAT30S D8
 U 1 1 5D64982C
 P 4700 1950
 F 0 "D8" H 4522 2071 50  0000 R CNN
 F 1 "D_BAT30S" H 4522 1980 50  0000 R CNN
-F 2 "" H 4700 1950 50  0001 C CNN
+F 2 "Package_TO_SOT_SMD:SOT-323_SC-70" H 4700 1950 50  0001 C CNN
 F 3 "" H 4700 1950 50  0001 C CNN
 	1    4700 1950
@@
 Wire Wire Line
 	7900 1550 7250 1550
-Wire Wire Line
-	4600 2150 4600 2250
 Connection ~ 7900 1550
 Wire Wire Line
@@
 	5650 1900 5600 1900
 $Comp
-L BAT30S:D_BAT30S D11
+L SAM21-rescue:D_BAT30S-BAT30S D11
 U 1 1 5D6570DE
 P 6600 1950
 F 0 "D11" H 6422 2071 50  0000 R CNN
 F 1 "D_BAT30S" H 6422 1980 50  0000 R CNN
-F 2 "" H 6600 1950 50  0001 C CNN
+F 2 "Package_TO_SOT_SMD:SOT-323_SC-70" H 6600 1950 50  0001 C CNN
 F 3 "" H 6600 1950 50  0001 C CNN
 	1    6600 1950
@@
 	1850 4200 2300 4200
 Text GLabel 1700 3800 0    50   Input ~ 0
-D14_I2C_PWR1.5C
+D14_I2C_PWR3.5B
 Wire Wire Line
 	1700 3800 1750 3800
@@
 	1750 3800 1850 3800
 Text GLabel 1550 4200 0    50   Input ~ 0
-D16_SCL1.5B
+D16_SCL3.5B
 Wire Wire Line
 	1550 4200 1850 4200
@@
 Connection ~ 3200 5000
 Text GLabel 1550 5000 0    50   Input ~ 0
-D15_SDA1.5B
+D15_SDA3.5B
 Wire Wire Line
 	1550 5000 1800 5000
@@
 	2750 6900 2750 6700
 Text GLabel 1450 6350 0    50   Input ~ 0
-D14_I2C_PWR1.5C
+D14_I2C_PWR3.5B
 Wire Wire Line
 	1450 6350 1650 6350
@@
 	9850 6100 9850 5900
 Text GLabel 8550 5550 0    50   Input ~ 0
-D9_UART_PWR1.5C
+D9_UART_PWR3.1D
 Wire Wire Line
 	8550 5550 8750 5550
@@
 	9450 1400 9300 1400
 Text GLabel 10300 1100 2    50   Input ~ 0
-D12_TX21.5C
+D12_TX23.3C
 Wire Wire Line
 	10300 1100 9800 1100
 Text GLabel 10300 1200 2    50   Input ~ 0
-D13_TX21.5C
+D13_RX23.3C
 Wire Wire Line
 	10300 1200 10100 1200
@@
 	9500 2450 9350 2450
 Text GLabel 10350 2150 2    50   Input ~ 0
-D10_TX11.5B
+D10_TX13.2C
 Wire Wire Line
 	10350 2150 9850 2150
 Text GLabel 10350 2250 2    50   Input ~ 0
-D11_RX11.5C
+D11_RX13.2C
 Wire Wire Line
 	10350 2250 10150 2250
@@
 	4700 1650 4700 1550
 $Comp
-L BAT30S:D_BAT30S D16
+L SAM21-rescue:D_BAT30S-BAT30S D16
 U 1 1 5D762A0A
 P 9200 3600
 F 0 "D16" H 9022 3721 50  0000 R CNN
 F 1 "D_BAT30S" H 9022 3630 50  0000 R CNN
-F 2 "" H 9200 3600 50  0001 C CNN
+F 2 "Package_TO_SOT_SMD:SOT-323_SC-70" H 9200 3600 50  0001 C CNN
 F 3 "" H 9200 3600 50  0001 C CNN
 	1    9200 3600
@@
 $EndComp
 $Comp
-L BAT30S:D_BAT30S D17
+L SAM21-rescue:D_BAT30S-BAT30S D17
 U 1 1 5D7633E5
 P 10100 3600
 F 0 "D17" H 9922 3721 50  0000 R CNN
 F 1 "D_BAT30S" H 9922 3630 50  0000 R CNN
-F 2 "" H 10100 3600 50  0001 C CNN
+F 2 "Package_TO_SOT_SMD:SOT-323_SC-70" H 10100 3600 50  0001 C CNN
 F 3 "" H 10100 3600 50  0001 C CNN
 	1    10100 3600
@@
 Connection ~ 10100 3200
 Text GLabel 10500 3550 2    50   Input ~ 0
-D12_TX21.5C
+D12_TX23.3C
 Wire Wire Line
 	10500 3550 10350 3550
 Text GLabel 9750 3900 2    50   Input ~ 0
-D13_TX21.5C
+D13_RX23.3C
 Wire Wire Line
 	9600 3550 9450 3550
@@
 UART
 $Comp
-L BAT30S:D_BAT30S D18
+L SAM21-rescue:D_BAT30S-BAT30S D18
 U 1 1 5D79CCE8
 P 6900 3850
 F 0 "D18" H 6722 3971 50  0000 R CNN
 F 1 "D_BAT30S" H 6722 3880 50  0000 R CNN
-F 2 "" H 6900 3850 50  0001 C CNN
+F 2 "Package_TO_SOT_SMD:SOT-323_SC-70" H 6900 3850 50  0001 C CNN
 F 3 "" H 6900 3850 50  0001 C CNN
 	1    6900 3850
@@
 $EndComp
 $Comp
-L BAT30S:D_BAT30S D19
+L SAM21-rescue:D_BAT30S-BAT30S D19
 U 1 1 5D79CCEE
 P 7800 3850
 F 0 "D19" H 7622 3971 50  0000 R CNN
 F 1 "D_BAT30S" H 7622 3880 50  0000 R CNN
-F 2 "" H 7800 3850 50  0001 C CNN
+F 2 "Package_TO_SOT_SMD:SOT-323_SC-70" H 7800 3850 50  0001 C CNN
 F 3 "" H 7800 3850 50  0001 C CNN
 	1    7800 3850
@@
 Connection ~ 7800 3450
 Text GLabel 8200 3800 2    50   Input ~ 0
-D10_TX11.5B
+D10_TX13.2C
 Wire Wire Line
 	8200 3800 8050 3800
 Text GLabel 7450 4150 2    50   Input ~ 0
-D11_RX11.5C
+D11_RX13.2C
 Wire Wire Line
 	7300 3800 7150 3800
@@
 	650  550  650  2950
 $Comp
-L DMP1045U:DMP1045U D23
+L SAM21-rescue:DMP1045U-DMP1045U D23
 U 1 1 5D5DDCBC
 P 2750 5900
@@
 	3250 6150 3250 6250
 $Comp
-L DMP1045U:DMP1045U D22
+L SAM21-rescue:DMP1045U-DMP1045U D22
 U 1 1 5D64C909
 P 9850 5000
@@
 Text Notes 2500 3700 0    118  ~ 24
 I2C
+$Comp
+L Mechanical:MountingHole H1
+U 1 1 5D4FC693
+P 5500 6400
+F 0 "H1" H 5600 6446 50  0000 L CNN
+F 1 "MountingHole" H 5600 6355 50  0000 L CNN
+F 2 "MountingHole:MountingHole_3.2mm_M3" H 5500 6400 50  0001 C CNN
+F 3 "~" H 5500 6400 50  0001 C CNN
+	1    5500 6400
+	1    0    0    -1
+$EndComp
+$Comp
+L Mechanical:MountingHole H2
+U 1 1 5D4FD480
+P 6200 6400
+F 0 "H2" H 6300 6446 50  0000 L CNN
+F 1 "MountingHole" H 6300 6355 50  0000 L CNN
+F 2 "MountingHole:MountingHole_3.2mm_M3" H 6200 6400 50  0001 C CNN
+F 3 "~" H 6200 6400 50  0001 C CNN
+	1    6200 6400
+	1    0    0    -1
+$EndComp
+$Comp
+L Mechanical:MountingHole H3
+U 1 1 5D4FD949
+P 5500 6700
+F 0 "H3" H 5600 6746 50  0000 L CNN
+F 1 "MountingHole" H 5600 6655 50  0000 L CNN
+F 2 "MountingHole:MountingHole_3.2mm_M3" H 5500 6700 50  0001 C CNN
+F 3 "~" H 5500 6700 50  0001 C CNN
+	1    5500 6700
+	1    0    0    -1
+$EndComp
+$Comp
+L Mechanical:MountingHole H4
+U 1 1 5D4FDB65
+P 6200 6700
+F 0 "H4" H 6300 6746 50  0000 L CNN
+F 1 "MountingHole" H 6300 6655 50  0000 L CNN
+F 2 "MountingHole:MountingHole_3.2mm_M3" H 6200 6700 50  0001 C CNN
+F 3 "~" H 6200 6700 50  0001 C CNN
+	1    6200 6700
+	1    0    0    -1
+$EndComp
+Wire Wire Line
+	4700 2150 4700 2100
 $EndSCHEMATC
