File: Power.sch (KiCad schematic (older format))
At the start: 10 parts, among them J3 Conn_01x02_Male, U2 AP1117-33

Commit message: Add files via upload
Parts:
- J3: footprint Connector_PinSocket_2.54mm:PinSocket_1x02_P2.54mm_Vertical -> Connector_JST:JST_EH_B2B-EH-A_1x02_P2.50mm_Vertical
Changed lines of the file:
@@
 F 0 "J3" H 2708 2931 50  0000 C CNN
 F 1 "Conn_01x02_Male" H 2708 2840 50  0000 C CNN
-F 2 "Connector_PinSocket_2.54mm:PinSocket_1x02_P2.54mm_Vertical" H 2600 2750 50  0001 C CNN
+F 2 "Connector_JST:JST_EH_B2B-EH-A_1x02_P2.50mm_Vertical" H 2600 2750 50  0001 C CNN
 F 3 "~" H 2600 2750 50  0001 C CNN
 	1    2600 2750
