File: XBee_Sockets.sch (KiCad schematic (older format))
At the start: 32 parts, among them Q1 BSS138, Q2 BSS138, U4 74lvc244, U5 XBEE, U7 XBEE

Commit message: Add files via upload
Parts:
- D20, D21: symbol DMP1045U:DMP1045U -> SAM21-rescue:DMP1045U-DMP1045U
- U4: symbol 74lvc244:74lvc244 -> SAM21-rescue:74lvc244-74lvc244
- U5, U7: symbol XBEE:XBEE -> SAM21-rescue:XBEE-XBEE
Connections:
- net XB2_MISO: no longer U4.9 (2Y3)
- net D19_MOSI1.5B renamed D19_MOSI2.2A
- net D20_SCK1.5B renamed D20_SCK2.2A
- net D21_MISO1.5B renamed D21_MISO2.2A
- net D22_XB1_PWR1.5C renamed D22_XB1_PWR2.5A
- net D23_CS_XB11.5 renamed D23_CS_XB12.2A
- net D24_INT_XB11.5B renamed D24_INT_XB12.4B
- net D25_TX_XB11.5C renamed D25_TX_XB12.2B
- net D26_RX_XB11.5C renamed D26_RX_XB12.2B
- net D27_XB2_PWR1.5C renamed D27_XB2_PWR2.5B
- net D28_CS_XB21.5 renamed D28_CS_XB22.2C
- net D29_INT_XB21.5B renamed D29_INT_XB22.4D
- net D30_TX_XB21.5B renamed D30_TX_XB22.2C
- net D31_RX_XB21.5B renamed D31_RX_XB22.2C
- new net D21_MISO2.3A: U4.9 (2Y3)
Changed lines of the file:
@@
 $EndDescr
 $Comp
-L 74lvc244:74lvc244 U4
+L SAM21-rescue:74lvc244-74lvc244 U4
 U 1 1 5D539CF4
 P 3250 2100
+AR Path="/5D539CF4" Ref="U4"  Part="1"
+AR Path="/5D5386B1/5D539CF4" Ref="U4"  Part="1"
 F 0 "U4" H 3250 2865 50  0000 C CNN
 F 1 "74lvc244" H 3250 2774 50  0000 C CNN
@@
 	1250 1550 1350 1550
 Text GLabel 1250 1850 0    50   Input ~ 0
-D23_CS_XB11.5
+D23_CS_XB12.2A
 Wire Wire Line
 	1250 1850 1650 1850
@@
 	1650 1850 1650 1750
 Text GLabel 2500 1700 0    50   Input ~ 0
-D19_MOSI1.5B
+D19_MOSI2.2A
 Text GLabel 2500 2000 0    50   Input ~ 0
-D20_SCK1.5B
+D20_SCK2.2A
 Text GLabel 2500 2300 0    50   Input ~ 0
 XB1_MISO
@@
 XB1_SCK
 Text GLabel 4050 2450 2    50   Input ~ 0
-D21_MISO1.5B
+D21_MISO2.2A
 Wire Wire Line
 	4050 2450 3850 2450
@@
 	5600 1100 5500 1100
 Text GLabel 5600 800  2    50   Input ~ 0
-D28_CS_XB21.5
+D28_CS_XB22.2C
 Wire Wire Line
 	5600 800  5200 800
@@
 	5200 1400 5200 1700
 Text GLabel 4050 2000 2    50   Input ~ 0
-D20_SCK1.5B
+D20_SCK2.2A
 Wire Wire Line
 	4050 2000 3850 2000
 Text GLabel 4050 2300 2    50   Input ~ 0
-D19_MOSI1.5B
+D19_MOSI2.2A
 Wire Wire Line
 	4050 2300 3850 2300
@@
 XB2_MOSI
 Text GLabel 2500 2450 0    50   Input ~ 0
-XB2_MISO
+D21_MISO2.3A
 Wire Wire Line
 	2500 2450 2650 2450
@@
 	4950 5550 4850 5550
 Text GLabel 4950 5550 2    50   Input ~ 0
-D24_INT_XB11.5B
+D24_INT_XB12.4B
 Wire Wire Line
 	4550 5550 4250 5550
@@
 XB1_MISO
 Text GLabel 1550 4950 0    50   Input ~ 0
-D25_TX_XB11.5C
+D25_TX_XB12.2B
 Text GLabel 1550 4850 0    50   Input ~ 0
-D26_RX_XB11.5C
+D26_RX_XB12.2B
 Wire Wire Line
 	1550 4750 2650 4750
@@
 XB1_VCC
 $Comp
-L XBEE:XBEE U5
+L SAM21-rescue:XBEE-XBEE U5
 U 1 1 5D566A6B
 P 3500 5150
@@
 	10450 5500 10350 5500
 Text GLabel 10450 5500 2    50   Input ~ 0
-D29_INT_XB21.5B
+D29_INT_XB22.4D
 Wire Wire Line
 	10050 5500 9750 5500
@@
 XB2_MISO
 Text GLabel 7050 4900 0    50   Input ~ 0
-D30_TX_XB21.5B
+D30_TX_XB22.2C
 Text GLabel 7050 4800 0    50   Input ~ 0
-D31_RX_XB21.5B
+D31_RX_XB22.2C
 Wire Wire Line
 	7050 4700 8150 4700
@@
 XB2_VCC
 $Comp
-L XBEE:XBEE U7
+L SAM21-rescue:XBEE-XBEE U7
 U 1 1 5D5AD446
 P 9000 5100
@@
 	8800 1350 9050 1350
 Text GLabel 8650 1350 0    50   Input ~ 0
-D22_XB1_PWR1.5C
+D22_XB1_PWR2.5A
 Wire Wire Line
 	8650 1350 8800 1350
@@
 	6300 2700 6550 2700
 Text GLabel 6150 2700 0    50   Input ~ 0
-D27_XB2_PWR1.5C
+D27_XB2_PWR2.5B
 Wire Wire Line
 	6150 2700 6300 2700
@@
 	6550 7350 6550 7150
 $Comp
-L DMP1045U:DMP1045U D20
+L SAM21-rescue:DMP1045U-DMP1045U D20
 U 1 1 5D4CF314
 P 9350 1450
@@
 $EndComp
 $Comp
-L DMP1045U:DMP1045U D21
+L SAM21-rescue:DMP1045U-DMP1045U D21
 U 1 1 5D4EC4FC
 P 6850 2800
