File: uC.sch (KiCad schematic (older format))
At the start: 30 parts, among them J1 614105150621, J2 Conn_01x05_Male, SW1 SW_DPST_x2, U1 ATSAMD21G18A-MU, U3 ESD5V3U2U-03F, U9 ATECC608A-MAHDA, Y1 32.768kHz

Commit message: Add files via upload
Parts:
- removed J1: 614105150621, 614105150621, symbol 614105150621:614105150621
- removed J2: Conn_01x05_Male, Connector_PinSocket_2.54mm:PinSocket_1x05_P2.54mm_Vertical, symbol Connector:Conn_01x05_Male
- removed SW1: SW_DPST_x2, Resistor_SMD:R_0402_1005Metric, symbol Switch:SW_DPST_x2
- added J1: 629105150521, microusb:microusb, symbol 629105150521:629105150521
- added J2: Conn_ARM_JTAG_SWD_10, Connector_PinHeader_1.27mm:PinHeader_2x05_P1.27mm_Vertical_SMD, symbol Connector:Conn_ARM_JTAG_SWD_10
- added SW1, SW2: SW_Push, Button_Switch_SMD:SW_SPST_EVPBF, symbol Switch:SW_Push
- L1: footprint (none) -> Inductor_SMD:L_0603_1608Metric
- U1: footprint QFN50P700X700X90-49N -> ATSAMD21G18A-MU:QFN50P700X700X90-49N; symbol ATSAMD21G18A-MU:ATSAMD21G18A-MU -> SAM21-rescue:ATSAMD21G18A-MU-ATSAMD21G18A-MU
- U3: symbol esd5v3u2u-03f:ESD5V3U2U-03F -> SAM21-rescue:ESD5V3U2U-03F-esd5v3u2u-03f
- U9: footprint (none) -> UDFN-8:UDFN-8; symbol ATECC608:ATECC608A-MAHDA -> SAM21-rescue:ATECC608A-MAHDA-ATECC608
- Y1: footprint (none) -> ECS-.327-12.5-34B-TR:XTAL_ECS-.327-12.5-34B-TR
Connections:
- net D17_SDA_IMU1.5B is gone; now on net D17_SDA_IMU4.3B: U9.5 (SDA)
- net D18_SCL_IMU1.5B is gone; now on net D18_SCL_IMU4.3B: U9.6 (SCL)
- net D7_STATUS_GREEN is gone; now on net D8_STATUS_GREEN: R6.2
- net VDDCORE is gone; now on net +3V3: C3.1, U1.43 (VDDCORE)
- net #RESET: now also J2.10 (~RESET~)
- net +3V3: now also J2.1 (VTref); no longer C10.1, F1.2
- net GND: now also U1.49 (EXP), J1.5 (GND), J2.3 (GND), J2.5 (GND), J2.9 (GNDDetect), SW1.2, SW2.1
- net SWCLK: now also J2.4 (SWDCLK/TCK)
- net SWDIO: now also J2.2 (SWDIO/TMS)
- net USB_D_N: now also J1.2 (D-)
- net USB_D_P: now also J1.3 (D+)
- net VBUS: now also J1.1 (VBUS)
- net at R1.1: now also J1.SHELL (SHIELD), J1.SHELL1 (SHIELD), J1.SHELL2 (SHIELD), J1.SHELL3 (SHIELD)
- net at R4.1: now also SW1.1
- net at R3.2: now also SW2.2
- net D20_5CK2.2A renamed D20_SCK2.2A
- new net +5V: C10.1, F1.2
- no-connect marks 5 -> 7
Other:
- moved on the sheet: R7
Changed lines of the file:
@@
 $EndDescr
 $Comp
-L ATSAMD21G18A-MU:ATSAMD21G18A-MU U1
+L SAM21-rescue:ATSAMD21G18A-MU-ATSAMD21G18A-MU U1
 U 1 1 5D3A8F5B
 P 6650 3250
 F 0 "U1" H 6650 5517 50  0000 C CNN
 F 1 "ATSAMD21G18A-MU" H 6650 5426 50  0000 C CNN
-F 2 "QFN50P700X700X90-49N" H 4750 1050 50  0001 L BNN
+F 2 "ATSAMD21G18A-MU:QFN50P700X700X90-49N" H 4750 1050 50  0001 L BNN
 F 3 "" H 4750 1200 50  0001 L BNN
 F 4 "QFN-48 Microchip" H 7500 2300 50  0001 L BNN "Field4"
@@
 F 0 "Y1" V 1704 5431 50  0000 L CNN
 F 1 "32.768kHz" V 1795 5431 50  0000 L CNN
-F 2 "" H 1750 5300 50  0001 C CNN
+F 2 "ECS-.327-12.5-34B-TR:XTAL_ECS-.327-12.5-34B-TR" H 1750 5300 50  0001 C CNN
 F 3 "~" H 1750 5300 50  0001 C CNN
 	1    1750 5300
@@
 F 0 "L1" V 10640 900 50  0000 C CNN
 F 1 "BLM18PG221SH1D" V 10549 900 50  0000 C CNN
-F 2 "" H 10450 900 50  0001 C CNN
+F 2 "Inductor_SMD:L_0603_1608Metric" H 10450 900 50  0001 C CNN
 F 3 "~" H 10450 900 50  0001 C CNN
 	1    10450 900
@@
 Wire Wire Line
 	7500 5250 7500 5150
-$Comp
-L 614105150621:614105150621 J1
-U 1 1 5D3BDB8F
-P 1100 2700
-F 0 "J1" H 1083 2110 50  0000 C CNN
-F 1 "614105150621" H 1083 2201 50  0000 C CNN
-F 2 "614105150621" H 1100 2700 50  0001 L BNN
-F 3 "" H 1100 2700 50  0001 L BNN
-F 4 "614105150621" H 1100 2700 50  0001 L BNN "Field4"
-F 5 "None" H 1100 2700 50  0001 L BNN "Field5"
-F 6 "Unavailable" H 1100 2700 50  0001 L BNN "Field6"
-F 7 "Wurth Electronics" H 1100 2700 50  0001 L BNN "Field7"
-F 8 "None" H 1100 2700 50  0001 L BNN "Field8"
-	1    1100 2700
-	-1   0    0    1
-$EndComp
 Text GLabel 3450 2700 2    50   Input ~ 0
 USB_D_P
@@
 Text GLabel 1950 3600 2    50   Input ~ 0
 VBUS
-$Comp
-L power:+3V3 #PWR010
-U 1 1 5D3C8BBB
-P 1200 3350
-F 0 "#PWR010" H 1200 3200 50  0001 C CNN
-F 1 "+3V3" H 1215 3523 50  0000 C CNN
-F 2 "" H 1200 3350 50  0001 C CNN
-F 3 "" H 1200 3350 50  0001 C CNN
-	1    1200 3350
-	1    0    0    -1
-$EndComp
 Wire Wire Line
 	1200 3350 1200 3600
@@
 	0    1    1    0
 $EndComp
-$Comp
-L Switch:SW_DPST_x2 SW1
-U 2 1 5D3D7F02
-P 6200 6300
-F 0 "SW1" H 6200 6535 50  0000 C CNN
-F 1 "SW_DPST_x2" H 6200 6444 50  0000 C CNN
-F 2 "Resistor_SMD:R_0402_1005Metric" H 6200 6300 50  0001 C CNN
-F 3 "~" H 6200 6300 50  0001 C CNN
-	2    6200 6300
-	1    0    0    -1
-$EndComp
 Wire Wire Line
 	6000 6300 5850 6300
@@
 	6550 7400 6300 7400
 Text GLabel 5400 7400 0    50   Input ~ 0
-D7_STATUS_GREEN
+D8_STATUS_GREEN
 Wire Wire Line
 	5400 7400 5500 7400
@@
 Wire Wire Line
 	3700 6250 4000 6250
-$Comp
-L Switch:SW_DPST_x2 SW1
-U 1 1 5D40C3E8
-P 3700 6950
-F 0 "SW1" V 3746 6862 50  0000 R CNN
-F 1 "SW_DPST_x2" V 3655 6862 50  0000 R CNN
-F 2 "Resistor_SMD:R_0402_1005Metric" H 3700 6950 50  0001 C CNN
-F 3 "~" H 3700 6950 50  0001 C CNN
-	1    3700 6950
-	0    -1   -1   0
-$EndComp
 Wire Wire Line
 	3700 6750 3700 6650
@@
 Wire Wire Line
 	3700 7150 3700 7300
-$Comp
-L Connector:Conn_01x05_Male J2
-U 1 1 5D413451
-P 900 6800
-F 0 "J2" H 1008 7181 50  0000 C CNN
-F 1 "Conn_01x05_Male" H 1008 7090 50  0000 C CNN
-F 2 "Connector_PinSocket_2.54mm:PinSocket_1x05_P2.54mm_Vertical" H 900 6800 50  0001 C CNN
-F 3 "~" H 900 6800 50  0001 C CNN
-	1    900  6800
-	1    0    0    -1
-$EndComp
-Text GLabel 1850 6600 2    50   Input ~ 0
+Text GLabel 3050 6600 2    50   Input ~ 0
 #RESET
-Text GLabel 1850 6700 2    50   Input ~ 0
+Text GLabel 3050 6900 2    50   Input ~ 0
 SWDIO
-Text GLabel 1850 6800 2    50   Input ~ 0
+Text GLabel 3050 6800 2    50   Input ~ 0
 SWCLK
 $Comp
 L power:GND #PWR020
 U 1 1 5D41D1D1
-P 1250 7050
-F 0 "#PWR020" H 1250 6800 50  0001 C CNN
-F 1 "GND" H 1255 6877 50  0000 C CNN
-F 2 "" H 1250 7050 50  0001 C CNN
-F 3 "" H 1250 7050 50  0001 C CNN
-	1    1250 7050
-	1    0    0    -1
-$EndComp
-Wire Wire Line
-	1250 7050 1250 7000
-Wire Wire Line
-	1250 7000 1100 7000
+P 2050 7600
+F 0 "#PWR020" H 2050 7350 50  0001 C CNN
+F 1 "GND" H 2055 7427 50  0000 C CNN
+F 2 "" H 2050 7600 50  0001 C CNN
+F 3 "" H 2050 7600 50  0001 C CNN
+	1    2050 7600
+	1    0    0    -1
+$EndComp
+Wire Wire Line
+	2050 7600 2050 7550
 $Comp
 L Device:R R7
 U 1 1 5D41FD41
-P 1350 6900
-F 0 "R7" V 1143 6900 50  0000 C CNN
-F 1 "1kE" V 1234 6900 50  0000 C CNN
-F 2 "Resistor_SMD:R_0402_1005Metric" V 1280 6900 50  0001 C CNN
-F 3 "~" H 1350 6900 50  0001 C CNN
-	1    1350 6900
+P 2150 6250
+F 0 "R7" V 1943 6250 50  0000 C CNN
+F 1 "1kE" V 2034 6250 50  0000 C CNN
+F 2 "Resistor_SMD:R_0402_1005Metric" V 2080 6250 50  0001 C CNN
+F 3 "~" H 2150 6250 50  0001 C CNN
+	1    2150 6250
 	0    1    1    0
 $EndComp
 Wire Wire Line
-	1100 6900 1200 6900
-Wire Wire Line
-	1100 6600 1850 6600
-Wire Wire Line
-	1100 6700 1850 6700
-Wire Wire Line
-	1100 6800 1700 6800
-Wire Wire Line
-	1500 6900 1700 6900
-Wire Wire Line
-	1700 6900 1700 6800
-Connection ~ 1700 6800
-Wire Wire Line
-	1700 6800 1850 6800
+	2300 6600 3050 6600
+Wire Wire Line
+	2300 6900 3050 6900
 $Comp
 L power:+3V3 #PWR019
 U 1 1 5D43160E
-P 1200 6450
-F 0 "#PWR019" H 1200 6300 50  0001 C CNN
-F 1 "+3V3" H 1215 6623 50  0000 C CNN
-F 2 "" H 1200 6450 50  0001 C CNN
-F 3 "" H 1200 6450 50  0001 C CNN
-	1    1200 6450
-	1    0    0    -1
-$EndComp
-Wire Wire Line
-	1200 6450 1200 6900
-Connection ~ 1200 6900
+P 1800 6150
+F 0 "#PWR019" H 1800 6000 50  0001 C CNN
+F 1 "+3V3" H 1815 6323 50  0000 C CNN
+F 2 "" H 1800 6150 50  0001 C CNN
+F 3 "" H 1800 6150 50  0001 C CNN
+	1    1800 6150
+	1    0    0    -1
+$EndComp
 Text GLabel 5800 2150 0    50   Input ~ 0
 D6_IO63.3B
@@
 D19_MOSI2.2A
 Text GLabel 5800 3650 0    50   Input ~ 0
-D20_5CK2.2A
+D20_SCK2.2A
 Text GLabel 5800 3750 0    50   Input ~ 0
 D23_CS_XB12.2A
@@
 	5800 3750 5950 3750
 $Comp
-L esd5v3u2u-03f:ESD5V3U2U-03F U3
+L SAM21-rescue:ESD5V3U2U-03F-esd5v3u2u-03f U3
 U 1 1 5D4FD829
 P 2750 3150
@@
 	2750 3550 2750 3650
 $Comp
-L ATECC608:ATECC608A-MAHDA U9
+L SAM21-rescue:ATECC608A-MAHDA-ATECC608 U9
 U 1 1 5D5E6491
 P 9100 5750
 F 0 "U9" H 9100 6215 50  0000 C CNN
 F 1 "ATECC608A-MAHDA" H 9100 6124 50  0000 C CNN
-F 2 "" H 9100 5750 50  0001 C CNN
+F 2 "UDFN-8:UDFN-8" H 9100 5750 50  0001 C CNN
 F 3 "" H 9100 5750 50  0001 C CNN
 	1    9100 5750
@@
 	10750 5450 10750 5550
 Text GLabel 9750 6000 2    50   Input ~ 0
-D17_SDA_IMU1.5B
+D17_SDA_IMU4.3B
 Text GLabel 9750 5850 2    50   Input ~ 0
-D18_SCL_IMU1.5B
+D18_SCL_IMU4.3B
 Wire Wire Line
 	9750 6000 9550 6000
@@
 Text Notes 9200 4950 0    118  ~ 24
 ATECC608A
+$Comp
+L 629105150521:629105150521 J1
+U 1 1 5D45FB94
+P 1100 2700
+F 0 "J1" H 1083 2110 50  0000 C CNN
+F 1 "629105150521" H 1083 2201 50  0000 C CNN
+F 2 "microusb:microusb" H 1100 2700 50  0001 L BNN
+F 3 "" H 1100 2700 50  0001 L BNN
+F 4 "Horizontal SMT Type B Version 2.0 MicroUSB Connector Socket, 30 V ac, 3A WR-COM" H 1100 2700 50  0001 L BNN "Field4"
+F 5 "None" H 1100 2700 50  0001 L BNN "Field5"
+F 6 "Wurth Electronics" H 1100 2700 50  0001 L BNN "Field6"
+F 7 "None" H 1100 2700 50  0001 L BNN "Field7"
+F 8 "Unavailable" H 1100 2700 50  0001 L BNN "Field8"
+	1    1100 2700
+	-1   0    0    1
+$EndComp
+$Comp
+L power:+5V #PWR0101
+U 1 1 5D453E63
+P 1200 3350
+F 0 "#PWR0101" H 1200 3200 50  0001 C CNN
+F 1 "+5V" H 1215 3523 50  0000 C CNN
+F 2 "" H 1200 3350 50  0001 C CNN
+F 3 "" H 1200 3350 50  0001 C CNN
+	1    1200 3350
+	1    0    0    -1
+$EndComp
+$Comp
+L Switch:SW_Push SW1
+U 1 1 5D455FDA
+P 6200 6300
+F 0 "SW1" H 6200 6585 50  0000 C CNN
+F 1 "SW_Push" H 6200 6494 50  0000 C CNN
+F 2 "Button_Switch_SMD:SW_SPST_EVPBF" H 6200 6500 50  0001 C CNN
+F 3 "~" H 6200 6500 50  0001 C CNN
+	1    6200 6300
+	1    0    0    -1
+$EndComp
+$Comp
+L Switch:SW_Push SW2
+U 1 1 5D45CF42
+P 3700 6950
+F 0 "SW2" V 3746 6902 50  0000 R CNN
+F 1 "SW_Push" V 3655 6902 50  0000 R CNN
+F 2 "Button_Switch_SMD:SW_SPST_EVPBF" H 3700 7150 50  0001 C CNN
+F 3 "~" H 3700 7150 50  0001 C CNN
+	1    3700 6950
+	0    -1   -1   0
+$EndComp
+$Comp
+L Connector:Conn_ARM_JTAG_SWD_10 J2
+U 1 1 5D58BACA
+P 1800 6900
+F 0 "J2" H 1357 6946 50  0000 R CNN
+F 1 "Conn_ARM_JTAG_SWD_10" H 1357 6855 50  0000 R CNN
+F 2 "Connector_PinHeader_1.27mm:PinHeader_2x05_P1.27mm_Vertical_SMD" H 1800 6900 50  0001 C CNN
+F 3 "http://infocenter.arm.com/help/topic/com.arm.doc.ddi0314h/DDI0314H_coresight_components_trm.pdf" V 1450 5650 50  0001 C CNN
+	1    1800 6900
+	1    0    0    -1
+$EndComp
+Wire Wire Line
+	1800 6150 1800 6250
+Wire Wire Line
+	2000 6250 1800 6250
+Connection ~ 1800 6250
+Wire Wire Line
+	1800 6250 1800 6300
+Wire Wire Line
+	2300 6800 2650 6800
+Wire Wire Line
+	1700 7550 1700 7500
+Wire Wire Line
+	1700 7550 1800 7550
+Wire Wire Line
+	1800 7500 1800 7550
+Connection ~ 1800 7550
+Wire Wire Line
+	1800 7550 2050 7550
+Wire Wire Line
+	2300 6250 2650 6250
+Wire Wire Line
+	2650 6250 2650 6800
+Connection ~ 2650 6800
+Wire Wire Line
+	2650 6800 3050 6800
+NoConn ~ 2300 7100
+NoConn ~ 2300 7000
+$Comp
+L power:+3V3 #PWR0102
+U 1 1 5D52CFED
+P 10500 1200
+F 0 "#PWR0102" H 10500 1050 50  0001 C CNN
+F 1 "+3V3" H 10515 1373 50  0000 C CNN
+F 2 "" H 10500 1200 50  0001 C CNN
+F 3 "" H 10500 1200 50  0001 C CNN
+	1    10500 1200
+	1    0    0    -1
+$EndComp
+Wire Wire Line
+	10500 1200 10500 1250
+Connection ~ 10500 1250
+Wire Wire Line
+	7350 5050 7500 5050
+Wire Wire Line
+	7500 5050 7500 5150
+Connection ~ 7500 5150
 $EndSCHEMATC
